File: BassPre.kicad_pcb (KiCad board)
At the start: 2 copper layers, 80 x 25 mm, 42 parts, among them P1 CONN_01X02, P2 CONN_01X02, P3 CONN_01X02, U1 TL072, U2 TL072, U3 TL072

Commit message: fix bypass capacitor position
Connections:
- C12 pad 2: Net-(C12-Pad2) -> GND
- P2 pad 2: Net-(C12-Pad2) -> Net-(P2-Pad2)
- P3 pad 1: Net-(C12-Pad2) -> Net-(P2-Pad2)
Routing:
- net Net-(C12-Pad2): track 11.8 -> 0.00 mm
- net GND: track 182.7 -> 192.7 mm
- net Net-(P2-Pad2): track 0.00 -> 5.08 mm
Other:
- board text added: "EQU01_v1.1 by M.S.T."
- board text removed: "EQU01_v1.0 by MST"
Changed lines of the file:
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@@
     (links 73)
     (no_connects 0)
-    (area 96.010714 47.389 183.989286 77.556)
+    (area 99.949999 49.949999 180.050001 75.050001)
     (thickness 1.6)
     (drawings 11)
-    (tracks 250)
+    (tracks 252)
     (zones 0)
     (modules 42)
@@
   (net 23 "Net-(R19-Pad1)")
   (net 24 "Net-(R16-Pad2)")
-  (net 25 "Net-(C12-Pad2)")
+  (net 25 "Net-(P2-Pad2)")
   (net_class Default "This is the default net class."
     (clearance 0.2)
@@
     (add_net "Net-(C11-Pad1)")
     (add_net "Net-(C11-Pad2)")
-    (add_net "Net-(C12-Pad2)")
     (add_net "Net-(C13-Pad1)")
     (add_net "Net-(C13-Pad2)")
@@
     (add_net "Net-(C7-Pad2)")
     (add_net "Net-(C9-Pad1)")
+    (add_net "Net-(P2-Pad2)")
     (add_net "Net-(R16-Pad2)")
     (add_net "Net-(R17-Pad1)")
@@
       (net 1 VCC))
     (pad 2 thru_hole oval (at 0 2.54 180) (size 1.7 1.7) (drill 1) (layers *.Cu *.Mask)
-      (net 25 "Net-(C12-Pad2)"))
+      (net 25 "Net-(P2-Pad2)"))
     (model ${KISYS3DMOD}/Pin_Headers.3dshapes/Pin_Header_Straight_1x02_Pitch2.54mm.wrl
       (at (xyz 0 0 0))
@@
     )
     (pad 1 thru_hole rect (at 0 0 180) (size 1.7 1.7) (drill 1) (layers *.Cu *.Mask)
-      (net 25 "Net-(C12-Pad2)"))
+      (net 25 "Net-(P2-Pad2)"))
     (pad 2 thru_hole oval (at 0 2.54 180) (size 1.7 1.7) (drill 1) (layers *.Cu *.Mask)
       (net 2 GND))
@@
       (net 1 VCC))
     (pad 2 smd rect (at 2.2 0 270) (size 3 1.6) (layers F.Cu F.Paste F.Mask)
-      (net 25 "Net-(C12-Pad2)"))
+      (net 2 GND))
     (model Capacitors_SMD.3dshapes/CP_Elec_5x5.3.wrl
       (at (xyz 0 0 0))
@@
   (gr_line (start 163.068 72.8218) (end 163.83 72.8218) (angle 90) (layer F.SilkS) (width 0.2))
   (gr_line (start 163.068 71.2978) (end 163.068 72.8218) (angle 90) (layer F.SilkS) (width 0.2))
-  (gr_text "EQU01_v1.0 by MST" (at 147.32 72.39) (layer F.SilkS)
+  (gr_text "EQU01_v1.1 by M.S.T." (at 145.5 72.5) (layer F.SilkS)
     (effects (font (size 1 1) (thickness 0.15)) (justify left))
   )
@@
   (segment (start 165.1 69.85) (end 163.83 71.12) (width 1) (layer F.Cu) (net 1))
   (segment (start 165.12 68.58) (end 162.56 68.58) (width 1) (layer F.Cu) (net 1))
+  (segment (start 170.18 53.34) (end 171.34 53.34) (width 0.25) (layer F.Cu) (net 2))
+  (segment (start 172 55) (end 176.53 59.53) (width 0.25) (layer F.Cu) (net 2))
+  (segment (start 172 54) (end 172 55) (width 0.25) (layer F.Cu) (net 2))
+  (segment (start 171.34 53.34) (end 172 54) (width 0.25) (layer F.Cu) (net 2))
+  (segment (start 176.53 59.53) (end 176.53 60.03) (width 0.25) (layer F.Cu) (net 2))
   (segment (start 172.72 68.5) (end 173.91 68.5) (width 0.25) (layer F.Cu) (net 2))
   (segment (start 177.8 67.31) (end 179.07 68.58) (width 0.25) (layer B.Cu) (net 2))
@@
   (segment (start 110.49 59.69) (end 110.49 67.31) (width 0.25) (layer B.Cu) (net 24))
   (segment (start 116.84 68.58) (end 114.3 71.12) (width 0.25) (layer F.Cu) (net 24))
-  (segment (start 170.18 60.96) (end 172.72 60.96) (width 0.25) (layer F.Cu) (net 25))
-  (segment (start 173.65 60.03) (end 176.53 60.03) (width 0.25) (layer F.Cu) (net 25))
-  (segment (start 172.72 60.96) (end 173.65 60.03) (width 0.25) (layer F.Cu) (net 25))
   (segment (start 170.18 60.96) (end 170.18 55.88) (width 1) (layer F.Cu) (net 25))
   (zone (net 2) (net_name GND) (layer B.Cu) (hatch edge 0.508)
